Commit message: + Save Commit from SaiK-7680!

File: wh_robot_urdf/urdf/robot_desc.xacro (robot description, xacro)
@@ -1,3 +1,7 @@
 <?xml version="1.0" encoding="utf-8"?>
-<robot name=>
+<robot name="warehouse_robot_desc" xmlns:xacro="http://www.ros.org/wiki/xacro">
+    <link name="world">
+    </link>
+    <xacro:include filename="$(find wh_robot_urdf)/urdf/robot_single.xacro">
+    <xacro:robot name="robot_1" parent="world" pos_x="1.0" pos_y="5.0"/>
 </robot>

Commit message: + Added simple robot and enabled visualization in RViz2!

File: wh_robot_urdf/urdf/robot_desc.xacro (robot description, xacro)
@@ -3,5 +3,5 @@
     <link name="world">
     </link>
-    <xacro:include filename="$(find wh_robot_urdf)/urdf/robot_single.xacro">
-    <xacro:robot name="robot_1" parent="world" pos_x="1.0" pos_y="5.0"/>
+    <xacro:include filename="$(find wh_robot_urdf)/urdf/robot_single.xacro"/>
+    <xacro:robot name="robot_1" parent="world" pos_x="1.0" pos_y="2.0"/>
 </robot>

File: wh_robot_urdf/urdf/robot_single.xacro (robot description, xacro)
@@ -1,13 +1,13 @@
+<?xml version="1.0"?>
 <!-- Add a basic shape to get the robot working -->
-<?xml version="1.0"?>
 <robot xmlns:xacro="http://www.ros.org/wiki/xacro">
-    <xacro:macro name="robot" params="name parent_link pos_x pos_y">
+    <xacro:macro name="robot" params="name parent pos_x pos_y">
         <link name="${name}">
             <visual>
                 <origin xyz="${pos_x} ${pos_y} 0" rpy="0.0 0.0 0.0"/>
                 <geometry>
-                <box size="0.4 0.4 0.4"/>
+                    <box size="0.4 0.4 0.1"/>
                 </geometry>
-                <material name="blue"/>
+                <!-- <material name="blue"/> -->
             </visual>
         </link>
